File: hardware/Production/SparkFun_IoT_RedBoard-ESP32_v01-Panel.brd (EAGLE design)
At the start: 246.1 x 248.9 mm, 2526 parts, among them J1 5.5x2.1mm Barrel, J101 USB C, J102 USB_SOLDER_PADS, J103 M10NO_SILK, J108 QWIIC_RIGHT_ANGLE, J109 MICRO-SD-PUSH-PUSH-EXT-PIN, J110 5.5x2.1mm Barrel, J117 USB C, J118 USB_SOLDER_PADS, J119 M10NO_SILK, J124 QWIIC_RIGHT_ANGLE, J125 MICRO-SD-PUSH-PUSH-EXT-PIN, J126 5.5x2.1mm Barrel, J13 QWIIC_RIGHT_ANGLE, J133 USB C, J134 USB_SOLDER_PADS, J135 M10NO_SILK, J140 QWIIC_RIGHT_ANGLE, J141 MICRO-SD-PUSH-PUSH-EXT-PIN, J142 5.5x2.1mm Barrel, J149 USB C, J15 MICRO-SD-PUSH-PUSH-EXT-PIN, J150 USB_SOLDER_PADS, J151 M10NO_SILK, J156 QWIIC_RIGHT_ANGLE, J157 MICRO-SD-PUSH-PUSH-EXT-PIN, J158 5.5x2.1mm Barrel, J165 USB C, J166 USB_SOLDER_PADS, J167 M10NO_SILK, J172 QWIIC_RIGHT_ANGLE, J173 MICRO-SD-PUSH-PUSH-EXT-PIN, J174 5.5x2.1mm Barrel, J181 USB C, J182 USB_SOLDER_PADS, J183 M10NO_SILK, J188 QWIIC_RIGHT_ANGLE, J189 MICRO-SD-PUSH-PUSH-EXT-PIN, J190 5.5x2.1mm Barrel, J2 USB C, J21 USB C, J22 USB_SOLDER_PADS, J23 M10NO_SILK, J28 QWIIC_RIGHT_ANGLE, J29 MICRO-SD-PUSH-PUSH-EXT-PIN, J3 USB_SOLDER_PADS, J30 5.5x2.1mm Barrel, J37 USB C, J38 USB_SOLDER_PADS, J39 M10NO_SILK, J44 QWIIC_RIGHT_ANGLE, J45 MICRO-SD-PUSH-PUSH-EXT-PIN, J46 5.5x2.1mm Barrel, J5 M10NO_SILK, J53 USB C, J54 USB_SOLDER_PADS, J55 M10NO_SILK, J60 QWIIC_RIGHT_ANGLE, J61 MICRO-SD-PUSH-PUSH-EXT-PIN, J62 5.5x2.1mm Barrel, J69 USB C, J70 USB_SOLDER_PADS, J71 M10NO_SILK, J76 QWIIC_RIGHT_ANGLE, J77 MICRO-SD-PUSH-PUSH-EXT-PIN, J78 5.5x2.1mm Barrel, J85 USB C, J86 USB_SOLDER_PADS, J87 M10NO_SILK, J92 QWIIC_RIGHT_ANGLE, J93 MICRO-SD-PUSH-PUSH-EXT-PIN, J94 5.5x2.1mm Barrel, Q1 MBT3904DW1T1, Q100 20V/4.2A/52mΩ/1.4W, Q102 20V/4.2A/52mΩ/1.4W, Q104 20V/4.2A/52mΩ/1.4W, Q105 MBT3904DW1T1, Q107 20V/4.2A/52mΩ/1.4W, Q109 20V/4.2A/52mΩ/1.4W, Q11 20V/4.2A/52mΩ/1.4W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

Commit message: Flipped Q3, added 100R resistor to Q3's gate and changed panel to 2x2 boards
Parts:
- removed BYP10, BYP11, BYP4, BYP5, BYP6, BYP7, BYP8, BYP9, JP108, JP122, JP136, JP150, JP164, JP66, JP80, JP94: JUMPER-SMT_2_NO_SILK, SparkFun-Jumpers:SMT-JUMPER_2_NO_SILK
- removed C100, C101, C117, C118, C134, C135, C151, C152, C168, C169, C185, C186, C202, C203, C83, C84: 4.7uF, SparkFun-Capacitors:0603
- removed C102, C103, C104, C107, C108, C109, C112, C114, C116, C119, C120, C121, C124, C125, C126, C129, C131, C133, C136, C137, C138, C141, C142, C143, C146, C148, C150, C153, C154, C155, C158, C159, C160, C163, C165, C167, C170, C171, C172, C175, C176, C177, C180, C182, C184, C187, C188, C189, C192, C193, C194, C197, C199, C201, C204, C69, C70, C73, C74, C75, C78, C80, C82, C85, C86, C87, C90, C91, C92, C95, C97, C99: 0.1uF, SparkFun-Capacitors:0603
- removed C105, C111, C122, C128, C139, C145, C156, C162, C173, C179, C190, C196, C71, C77, C88, C94: 10uF, SparkFun-Capacitors:EIA3216
- removed C106, C123, C140, C157, C174, C191, C72, C89: 10nF, SparkFun-Capacitors:0603
- removed C110, C115, C127, C132, C144, C149, C161, C166, C178, C183, C195, C200, C76, C81, C93, C98: 10uF, SparkFun-Capacitors:0603
- removed C113, C130, C147, C164, C181, C198, C79, C96: 47uF, SparkFun-Capacitors:PANASONIC_D
- removed D25, D31, D37, D43, D49, D55, D61, D67: GREEN, SparkFun-LED:LED-1206-HIDDENSILK
- removed D26, D32, D38, D44, D50, D56, D62, D68: YELLOW, SparkFun-LED:LED-1206-HIDDENSILK
- removed D27, D33, D39, D45, D51, D57, D63, D69: BLUE, SparkFun-LED:LED-1206-HIDDENSILK
- removed D28, D34, D40, D46, D52, D58, D64, D70: 1A/40V/500mV, SparkFun-DiscreteSemi:SMA-DIODE
- removed D29, D35, D41, D47, D53, D59, D65, D71: RED, SparkFun-LED:LED-1206-HIDDENSILK
- removed D30, D36, D42, D48, D54, D60, D66, D72: PWR, SparkFun-LED:LED-1206-HIDDENSILK
- removed F10, F11, F12, F5, F6, F7, F8, F9: 6V/2A, SparkFun-Fuses:1210
- removed J100, J116, J132, J148, J164, J180, J68, J84: (no value), SparkFun-Connectors:1X06_SMD_STRAIGHT_COMBO
- removed J101, J117, J133, J149, J165, J181, J69, J85: USB C, SparkFun-Connectors:USB-C-16P-2LAYER-PADS
- removed J102, J118, J134, J150, J166, J182, J70, J86: USB_SOLDER_PADS, SparkFun-Connectors:USB-SOLDER-PADS
- removed J103, J119, J135, J151, J167, J183, J71, J87: M10NO_SILK, SparkFun-Connectors:1X10_NO_SILK
- removed J104, J106, J120, J122, J136, J138, J152, J154, J168, J170, J184, J186, J72, J74, J88, J90: (no value), SparkFun-Connectors:1X08_NO_SILK
- removed J105, J121, J137, J153, J169, J185, J73, J89: (no value), SparkFun-Connectors:1X06_NO_SILK
- removed J107, J123, J139, J155, J171, J187, J75, J91: (no value), SparkFun-Connectors:2X5_PTH_SILK_.05
- removed J108, J124, J140, J156, J172, J188, J76, J92: QWIIC_RIGHT_ANGLE, SparkFun-Connectors:JST04_1MM_RA
- removed J109, J125, J141, J157, J173, J189, J77, J93: MICRO-SD-PUSH-PUSH-EXT-PIN, SparkFun-Connectors:MICROSD-EXTERNALPIN
- removed J110, J126, J142, J158, J174, J190, J78, J94: 5.5x2.1mm Barrel, SparkFun-Connectors:POWER_JACK_SMD
- removed J111, J112, J127, J128, J143, J144, J159, J160, J175, J176, J191, J192, J79, J80, J95, J96: (no value), SparkFun-Connectors:1X02_NO_SILK
- removed J113, J129, J145, J161, J177, J65, J81, J97: (no value), SparkFun-Connectors:1X10_SMD_COMBINED
- removed J114, J115, J130, J131, J146, J147, J162, J163, J178, J179, J66, J67, J82, J83, J98, J99: (no value), SparkFun-Connectors:1X08_SMD_COMBINED
- removed JP100, JP101, JP102, JP113, JP114, JP115, JP116, JP127, JP128, JP129, JP130, JP141, JP142, JP143, JP144, JP155, JP156, JP157, JP158, JP57, JP58, JP59, JP60, JP71, JP72, JP73, JP74, JP85, JP86, JP87, JP88, JP99: STAND-OFF, SparkFun-Hardware:STAND-OFF
- removed JP103, JP104, JP105, JP106, JP117, JP118, JP119, JP120, JP131, JP132, JP133, JP134, JP145, JP146, JP147, JP148, JP159, JP160, JP161, JP162, JP61, JP62, JP63, JP64, JP75, JP76, JP77, JP78, JP89, JP90, JP91, JP92: FIDUCIAL1X2, SparkFun-Aesthetics:FIDUCIAL-1X2
- removed JP107, JP121, JP135, JP149, JP163, JP65, JP79, JP93: JUMPER-SMT_3_2-NC_TRACE_SILK, SparkFun-Jumpers:SMT-JUMPER_3_2-NC_TRACE_SILK
- removed JP109, JP110, JP112, JP123, JP124, JP126, JP137, JP138, JP140, JP151, JP152, JP154, JP165, JP166, JP168, JP67, JP68, JP70, JP81, JP82, JP84, JP95, JP96, JP98: JUMPER-SMT_2_NC_TRACE_SILK, SparkFun-Jumpers:SMT-JUMPER_2_NC_TRACE_SILK
- removed JP111, JP125, JP139, JP153, JP167, JP69, JP83, JP97: LiPo, SparkFun-Connectors:JST-2-SMD
- removed LOGO17, LOGO21, LOGO25, LOGO29, LOGO33, LOGO37, LOGO41, LOGO45: SFE_LOGO_NAME.1_INCH, SparkFun-Aesthetics:SFE_LOGO_NAME_.1
- removed LOGO18, LOGO22, LOGO26, LOGO30, LOGO34, LOGO38, LOGO42, LOGO46: QWIIC_LOGO_5MM, SparkFun-Aesthetics:QWIIC_5MM
- removed LOGO19, LOGO23, LOGO27, LOGO31, LOGO35, LOGO39, LOGO43, LOGO47: OSHW-LOGOMINI, SparkFun-Aesthetics:OSHW-LOGO-MINI
- removed LOGO20, LOGO24, LOGO28, LOGO32, LOGO36, LOGO40, LOGO44, LOGO48: SFE_LOGO_NAME_FLAME.2_INCH, SparkFun-Aesthetics:SFE_LOGO_NAME_FLAME_.2
- removed Q100, Q102, Q104, Q107, Q109, Q111, Q113, Q115, Q117, Q120, Q122, Q124, Q126, Q128, Q130, Q133, Q135, Q137, Q139, Q141, Q143, Q146, Q148, Q150, Q152, Q154, Q156, Q55, Q57, Q59, Q61, Q63, Q65, Q68, Q70, Q72, Q74, Q76, Q78, Q81, Q83, Q85, Q87, Q89, Q91, Q94, Q96, Q98: 20V/4.2A/52mΩ/1.4W, SparkFun-DiscreteSemi:SOT23-3
- removed Q101, Q103, Q106, Q110, Q112, Q114, Q116, Q119, Q123, Q125, Q127, Q129, Q132, Q136, Q138, Q140, Q142, Q145, Q149, Q151, Q153, Q155, Q54, Q58, Q60, Q62, Q64, Q67, Q71, Q73, Q75, Q77, Q80, Q84, Q86, Q88, Q90, Q93, Q97, Q99: (no value), SparkFun-DiscreteSemi:SOT363_PHILIPS
- removed Q105, Q118, Q131, Q144, Q53, Q66, Q79, Q92: MBT3904DW1T1, SparkFun-DiscreteSemi:SC70-6
- removed Q108, Q121, Q134, Q147, Q56, Q69, Q82, Q95: (no value), SparkFun-DiscreteSemi:SC70-6
- removed R121, R122, R123, R129, R131, R132, R133, R134, R136, R140, R142, R144, R145, R150, R151, R152, R158, R160, R161, R162, R163, R165, R169, R171, R173, R174, R179, R180, R181, R187, R189, R190, R191, R192, R194, R198, R200, R202, R203, R208, R209, R210, R216, R218, R219, R220, R221, R223, R227, R229, R231, R232, R237, R238, R239, R245, R247, R248, R249, R250, R252, R256, R258, R260, R261, R266, R267, R268, R274, R276, R277, R278, R279, R281, R285, R287, R289, R290, R295, R296, R297, R303, R305, R306, R307, R308, R310, R314, R316, R318, R319, R324, R325, R326, R332, R334, R335, R336, R337, R339, R343, R345, R347, R348: 10k, SparkFun-Resistors:0603
- removed R124, R146, R147, R153, R175, R176, R182, R204, R205, R211, R233, R234, R240, R262, R263, R269, R291, R292, R298, R320, R321, R327: 4.7k, SparkFun-Resistors:0603
- removed R125, R126, R154, R155, R183, R184, R212, R213, R241, R242, R270, R271, R299, R300, R328, R329: 2.2k, SparkFun-Resistors:0603
- removed R127, R156, R185, R214, R243, R272, R301, R330: 715, SparkFun-Resistors:0603
- removed R128, R157, R186, R215, R244, R273, R302, R331: 240, SparkFun-Resistors:0603
- removed R130, R135, R137, R141, R143, R159, R164, R166, R170, R172, R188, R193, R195, R199, R201, R217, R222, R224, R228, R230, R246, R251, R253, R257, R259, R275, R280, R282, R286, R288, R304, R309, R311, R315, R317, R333, R338, R340, R344, R346: 47k, SparkFun-Resistors:0603
- removed R138, R167, R196, R225, R254, R283, R312, R341: 1k, SparkFun-Resistors:0603
- removed R139, R168, R197, R226, R255, R284, R313, R342: 2.0k, SparkFun-Resistors:0603
- removed R148, R149, R177, R178, R206, R207, R235, R236, R264, R265, R293, R294, R322, R323: 5.1k, SparkFun-Resistors:0603
- removed S10, S12, S14, S16, S18, S20, S22, S24: GPIO0, SparkFun-Switches:TACTILE_SWITCH_SMD_5.2MM
- removed S11, S13, S15, S17, S19, S21, S23, S9: Reset, SparkFun-Switches:TACTILE_SWITCH_SMD_5.2MM
- removed TP10, TP11, TP12, TP5, TP6, TP7, TP8, TP9: TEST-POINT3, SparkFun-Connectors:PAD.03X.03
- removed U$1000, U$1100, U$1200, U$500, U$600, U$700, U$800, U$900: (no value), output-ESP32:3#3V_LOGIC_SHIELDS_ONLY132321876
- removed U$1001, U$1101, U$401, U$501, U$601, U$701, U$801, U$901: (no value), output-ESP32:V323252
- removed U$1002, U$1102, U$402, U$502, U$602, U$702, U$802, U$902: (no value), output-ESP32:#SCL#34
- removed U$1003, U$1103, U$403, U$503, U$603, U$703, U$803, U$903: (no value), output-ESP32:#SDA#33
- removed U$1004, U$1104, U$404, U$504, U$604, U$704, U$804, U$904: (no value), output-ESP32:#3#3V#33
- removed U$1005, U$1105, U$405, U$505, U$605, U$705, U$805, U$905: (no value), output-ESP32:#GND#32
- removed U$1006, U$1106, U$406, U$506, U$606, U$706, U$806, U$906: (no value), output-ESP32:#SCK#31
- removed U$1007, U$1107, U$407, U$507, U$607, U$707, U$807, U$907: (no value), output-ESP32:#POCI#30
- removed U$1008, U$1108, U$408, U$508, U$608, U$708, U$808, U$908: (no value), output-ESP32:#PICO#29
- removed U$1009, U$1109, U$409, U$509, U$609, U$709, U$809, U$909: (no value), output-ESP32:1836
- removed U$1010, U$1110, U$410, U$510, U$610, U$710, U$810, U$910: (no value), output-ESP32:##CS##28
- removed U$1011, U$1111, U$411, U$511, U$611, U$711, U$811, U$911: (no value), output-ESP32:#27#27
- removed U$1012, U$1112, U$412, U$512, U$612, U$712, U$812, U$912: (no value), output-ESP32:#26#26
- removed U$1013, U$1113, U$413, U$513, U$613, U$713, U$813, U$913: (no value), output-ESP32:TX1838
- removed U$1014, U$1114, U$414, U$514, U$614, U$714, U$814, U$914: (no value), output-ESP32:RX1839
- removed U$1015, U$1115, U$415, U$515, U$615, U$715, U$815, U$915: (no value), output-ESP32:PWR1837
- removed U$1016, U$1116, U$416, U$516, U$616, U$716, U$816, U$916: (no value), output-ESP32:CHG1840
- removed U$1017, U$1117, U$417, U$517, U$617, U$717, U$817, U$917: (no value), output-ESP32:#25#18
- removed U$1018, U$1118, U$418, U$518, U$618, U$718, U$818, U$918: (no value), output-ESP32:#17#17
- removed U$1019, U$1119, U$419, U$519, U$619, U$719, U$819, U$919: (no value), output-ESP32:#16#15
- removed U$1020, U$1120, U$420, U$520, U$620, U$720, U$820, U$920: (no value), output-ESP32:#14#14
- removed U$1021, U$1121, U$421, U$521, U$621, U$721, U$821, U$921: (no value), output-ESP32:#13#5
- removed U$1022, U$1122, U$422, U$522, U$622, U$722, U$822, U$922: (no value), output-ESP32:#4#2
- removed U$1023, U$1123, U$423, U$523, U$623, U$723, U$823, U$923: (no value), output-ESP32:#TX#O#0
- removed U$1024, U$1124, U$424, U$524, U$624, U$724, U$824, U$924: (no value), output-ESP32:#RX#I#1
- removed U$1025, U$1125, U$425, U$525, U$625, U$725, U$825, U$925: (no value), output-ESP32:#RESET#1842
- removed U$1026, U$1126, U$426, U$526, U$626, U$726, U$826, U$926: (no value), output-ESP32:#BOOT#1841
- removed U$1027, U$1045, U$1127, U$1145, U$427, U$445, U$527, U$545, U$627, U$645, U$727, U$745, U$827, U$845, U$927, U$945: (no value), output-ESP32:#JTAG#1847
- removed U$1028, U$1128, U$428, U$528, U$628, U$728, U$828, U$928: (no value), output-ESP32:#A0#1843
- removed U$1029, U$1129, U$429, U$529, U$629, U$729, U$829, U$929: (no value), output-ESP32:#A3#1843
- removed U$1030, U$1130, U$430, U$530, U$630, U$730, U$830, U$930: (no value), output-ESP32:#A6#1843
- removed U$1031, U$1131, U$431, U$531, U$631, U$731, U$831, U$931: (no value), output-ESP32:#A7#1843
- removed U$1032, U$1132, U$432, U$532, U$632, U$732, U$832, U$932: (no value), output-ESP32:#A4#1843
- removed U$1033, U$1133, U$433, U$533, U$633, U$733, U$833, U$933: (no value), output-ESP32:#A5#1843
- removed U$1034, U$1134, U$434, U$534, U$634, U$734, U$834, U$934: (no value), output-ESP32:#VIN#1843
- removed U$1035, U$1036, U$1135, U$1136, U$435, U$436, U$535, U$536, U$635, U$636, U$735, U$736, U$835, U$836, U$935, U$936: (no value), output-ESP32:#GND#1844
- removed U$1037, U$1137, U$437, U$537, U$637, U$737, U$837, U$937: (no value), output-ESP32:#5V#1845
- removed U$1038, U$1138, U$438, U$538, U$638, U$738, U$838, U$938: (no value), output-ESP32:#3#3V#1845
- removed U$1039, U$1139, U$439, U$539, U$639, U$739, U$839, U$939: (no value), output-ESP32:##RST##1845
- removed U$1040, U$1140, U$440, U$540, U$640, U$740, U$840, U$940: (no value), output-ESP32:#REF#1846
- removed U$1041, U$1078, U$1141, U$1178, U$441, U$478, U$541, U$578, U$641, U$678, U$741, U$778, U$841, U$878, U$941, U$978: (no value), output-ESP32:#MEAS#1851
- removed U$1042, U$1083, U$1142, U$1183, U$442, U$483, U$542, U$583, U$642, U$683, U$742, U$783, U$842, U$883, U$942, U$983: (no value), output-ESP32:#1849
- removed U$1043, U$1084, U$1143, U$1184, U$443, U$484, U$543, U$584, U$643, U$684, U$743, U$784, U$843, U$884, U$943, U$984: (no value), output-ESP32:#1850
- removed U$1044, U$1144, U$444, U$544, U$644, U$744, U$844, U$944: (no value), output-ESP32:#BATT#1848
- removed U$1046, U$1146, U$446, U$546, U$646, U$746, U$846, U$946: (no value), output-ESP32:ESP321855
- removed U$1047, U$1099, U$1147, U$1199, U$447, U$499, U$547, U$599, U$647, U$699, U$747, U$799, U$847, U$899, U$947, U$999: (no value), output-ESP32:7#15V32321861
- removed U$1048, U$1148, U$448, U$548, U$648, U$748, U$848, U$948: (no value), output-ESP32:#39#A3#321862
- removed U$1049, U$1149, U$449, U$549, U$649, U$749, U$849, U$949: (no value), output-ESP32:#36#A0#321862
- removed U$1050, U$1150, U$450, U$550, U$650, U$750, U$850, U$950: (no value), output-ESP32:#34#A6#32321865
- removed U$1051, U$1151, U$451, U$551, U$651, U$751, U$851, U$951: (no value), output-ESP32:#35#A7#321862
- removed U$1052, U$1152, U$452, U$552, U$652, U$752, U$852, U$952: (no value), output-ESP32:#32#A4#32321865
- removed U$1053, U$1153, U$453, U$553, U$653, U$753, U$853, U$953: (no value), output-ESP32:#34#A6#321862
- removed U$1054, U$1154, U$454, U$554, U$654, U$754, U$854, U$954: (no value), output-ESP32:#VIN#321862
- removed U$1055, U$1058, U$1155, U$1158, U$455, U$458, U$555, U$558, U$655, U$658, U$755, U$758, U$855, U$858, U$955, U$958: (no value), output-ESP32:#GND#321863
- removed U$1056, U$1156, U$456, U$556, U$656, U$756, U$856, U$956: (no value), output-ESP32:#5V#321864
- removed U$1057, U$1157, U$457, U$557, U$657, U$757, U$857, U$957: (no value), output-ESP32:#3#3V#321864
- removed U$1059, U$1159, U$459, U$559, U$659, U$759, U$859, U$959: (no value), output-ESP32:##RESET##321864
- removed U$1060, U$1160, U$460, U$560, U$660, U$760, U$860, U$960: (no value), output-ESP32:#IOREF#321865
- removed U$1061, U$1161, U$461, U$561, U$661, U$761, U$861, U$961: (no value), output-ESP32:#3#RX#I#32321869
- removed U$1062, U$1162, U$462, U$562, U$662, U$762, U$862, U$962: (no value), output-ESP32:#1#TX#O#32321869
- removed U$1063, U$1163, U$463, U$563, U$663, U$763, U$863, U$963: (no value), output-ESP32:#13#TCK#32321869
- removed U$1064, U$1164, U$464, U$564, U$664, U$764, U$864, U$964: (no value), output-ESP32:#14#TMS#32321869
- removed U$1065, U$1165, U$465, U$565, U$665, U$765, U$865, U$965: (no value), output-ESP32:#16#32321869
- removed U$1066, U$1166, U$466, U$566, U$666, U$766, U$866, U$966: (no value), output-ESP32:#17#32321869
- removed U$1067, U$1167, U$467, U$567, U$667, U$767, U$867, U$967: (no value), output-ESP32:#25#32321869
- removed U$1068, U$1168, U$468, U$568, U$668, U$768, U$868, U$968: (no value), output-ESP32:#26#32321869
- removed U$1069, U$1169, U$469, U$569, U$669, U$769, U$869, U$969: (no value), output-ESP32:#5##CS##32321869
- removed U$1070, U$1170, U$470, U$570, U$670, U$770, U$870, U$970: (no value), output-ESP32:#23#PICO#321866
- removed U$1071, U$1171, U$471, U$571, U$671, U$771, U$871, U$971: (no value), output-ESP32:#19#POCI#321866
- removed U$1072, U$1172, U$472, U$572, U$672, U$772, U$872, U$972: (no value), output-ESP32:#18#SCK#32321869
- removed U$1073, U$1173, U$473, U$573, U$673, U$773, U$873, U$973: (no value), output-ESP32:#21#SDA#32321869
- removed U$1074, U$1174, U$474, U$574, U$674, U$774, U$874, U$974: (no value), output-ESP32:#22#SCL#32321869
- removed U$1075, U$1175, U$475, U$575, U$675, U$775, U$875, U$975: (no value), output-ESP32:#27#32321869
- removed U$1076, U$1176, U$476, U$576, U$676, U$776, U$876, U$976: (no value), output-ESP32:#GND#321866
- removed U$1077, U$1177, U$477, U$577, U$677, U$777, U$877, U$977: (no value), output-ESP32:#3#3V#321866
- removed U$1079, U$1179, U$479, U$579, U$679, U$779, U$879, U$979: (no value), output-ESP32:#BYP#35
- removed U$1080, U$1180, U$480, U$580, U$680, U$780, U$880, U$980: (no value), output-ESP32:D#32321863
- removed U$1081, U$1181, U$481, U$581, U$681, U$781, U$881, U$981: (no value), output-ESP32:D#32321862
- removed U$1082, U$1182, U$482, U$582, U$682, U$782, U$882, U$982: (no value), output-ESP32:G32321864
- removed U$1085, U$1185, U$485, U$585, U$685, U$785, U$885, U$985: (no value), output-ESP32:#I2C#1855
- removed U$1086, U$1186, U$486, U$586, U$686, U$786, U$886, U$986: (no value), output-ESP32:##ALERT##1852
- removed U$1087, U$1187, U$487, U$587, U$687, U$787, U$887, U$987: (no value), output-ESP32:#TMS#1854
- removed U$1088, U$1188, U$488, U$588, U$688, U$788, U$888, U$988: (no value), output-ESP32:#TCK#1853
- removed U$1089, U$1090, U$1189, U$1190, U$489, U$490, U$589, U$590, U$689, U$690, U$789, U$790, U$889, U$890, U$989, U$990: (no value), output-ESP32:INPUT_ONLY321867
- removed U$1091, U$1191, U$491, U$591, U$691, U$791, U$891, U$991: (no value), output-ESP32:##ALERT##4#321866
- removed U$1092, U$1192, U$492, U$592, U$692, U$792, U$892, U$992: (no value), output-ESP32:TP1321868
- removed U$1093, U$1193, U$493, U$593, U$693, U$793, U$893, U$993: (no value), SparkFun-Aesthetics:REDBOARD_LOGO
- removed U$1094, U$1194, U$494, U$594, U$694, U$794, U$894, U$994: (no value), output-ESP32:#IOT#132321869
- removed U$1095, U$1195, U$495, U$595, U$695, U$795, U$895, U$995: (no value), output-ESP32:ESP32321856
- removed U$1096, U$1196, U$496, U$596, U$696, U$796, U$896, U$996: (no value), output-ESP32:#IOT#132321874
- removed U$1097, U$1197, U$497, U$597, U$697, U$797, U$897, U$997: (no value), output-ESP32:MADE_IN32321857
- removed U$1098, U$1198, U$498, U$598, U$698, U$798, U$898, U$998: (no value), output-ESP32:THE_USA32321858
- removed U25, U31, U37, U43, U49, U55, U61, U67: CH340C, SparkFun-IC-Comms:SO016
- removed U26, U32, U38, U44, U50, U56, U62, U68: ESP-WROOM-3232D-NARROW, SparkFun-RF:ESP-WROOM-32D-NARROW
- removed U27, U33, U39, U45, U51, U57, U63, U69: LM1117, SparkFun-IC-Power:SOT223
- removed U28, U34, U40, U46, U52, U58, U64, U70: 3.3V, SparkFun-IC-Power:SOT23-5
- removed U29, U35, U41, U47, U53, U59, U65, U71: MCP73831, SparkFun-IC-Power:SOT23-5
- removed U30, U36, U42, U48, U54, U60, U66, U72: MAX17048, SparkFun-IC-Power:DFN-8
- R100: value 10k -> 2.2k
- R101: value 47k -> 715
- R102, R42: value 10k -> 240
- R104, R111, R115, R44, R49, R55, R57, R74, R87: value 10k -> 47k
- R106, R108, R114, R43, R48, R50, R54, R56, R77: value 47k -> 10k
- R109, R51: value 1k -> 47k
- R110: value 2.0k -> 10k
- R112: value 47k -> 1k
- R113, R53: value 10k -> 2.0k
- R117: value 4.7k -> 47k
- R118, R37, R59, R66, R88, R89, R95: value 4.7k -> 10k
- R119: value 5.1k -> 10k
- R120, R90: value 5.1k -> 100
- R30, R60: value 4.7k -> 100
- R32, R61, R62, R91: value 5.1k -> 4.7k
- R34, R63, R64, R93, R94: value 10k -> 5.1k
- R38, R68: value 2.2k -> 4.7k
- R40, R69: value 715 -> 2.2k
- R41: value 240 -> 715
- R52: value 2.0k -> 1k
- R67, R96, R97: value 2.2k -> 10k
- R70, R99: value 240 -> 2.2k
- R71: value 10k -> 715
- R72: value 47k -> 240
- R80: value 1k -> 10k
- R81: value 2.0k -> 47k
- R82: value 10k -> 1k
- R83: value 47k -> 2.0k
- R92: value 10k -> 4.7k
- R98: value 715 -> 4.7k
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Connections:
- removed net !DTR!10: Q131.4, R296.1, U61.13
- removed net !DTR!11: Q144.4, R325.1, U67.13
- removed net !DTR!4: Q53.4, R122.1, U25.13
- removed net !DTR!5: Q66.4, R151.1, U31.13
- removed net !DTR!6: Q79.4, R180.1, U37.13
- removed net !DTR!7: Q92.4, R209.1, U43.13
- removed net !DTR!8: Q105.4, R238.1, U49.13
- removed net !DTR!9: Q118.4, R267.1, U55.13
- removed net !GAUGE_ALERT!10: JP150.1, R318.1, U66.5
- removed net !GAUGE_ALERT!11: JP164.1, R347.1, U72.5
- removed net !GAUGE_ALERT!4: JP66.1, R144.1, U30.5
- removed net !GAUGE_ALERT!5: JP80.1, R173.1, U36.5
- removed net !GAUGE_ALERT!6: JP94.1, R202.1, U42.5
- removed net !GAUGE_ALERT!7: JP108.1, R231.1, U48.5
- removed net !GAUGE_ALERT!8: JP122.1, R260.1, U54.5
- removed net !GAUGE_ALERT!9: JP136.1, R289.1, U60.5
- removed net !RTS!10: Q131.1, R295.1, U61.14
- removed net !RTS!11: Q144.1, R324.1, U67.14
- removed net !RTS!4: Q53.1, R121.1, U25.14
- removed net !RTS!5: Q66.1, R150.1, U31.14
- removed net !RTS!6: Q79.1, R179.1, U37.14
- removed net !RTS!7: Q92.1, R208.1, U43.14
- removed net !RTS!8: Q105.1, R237.1, U49.14
- removed net !RTS!9: Q118.1, R266.1, U55.14
- removed net 3.3V10: C175.1, C177.1, C178.1, C182.1, C183.1, D61.A, D62.A, D66.A, J161.3A, J161.3B, J162.2, J162.4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
- removed net 3.3V11: C192.1, C194.1, C195.1, C199.1, C200.1, D67.A, D68.A, D72.A, J177.3A, J177.3B, J178.2, J178.4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
- removed net 3.3V4: C73.1, C75.1, C76.1, C80.1, C81.1, D25.A, D26.A, D30.A, J65.3A, J65.3B, J66.2, J66.4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
- removed net 3.3V5: C90.1, C92.1, C93.1, C97.1, C98.1, D31.A, D32.A, D36.A, J81.3A, J81.3B, J82.2, J82.4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
- removed net 3.3V6: C107.1, C109.1, C110.1, C114.1, C115.1, D37.A, D38.A, D42.A, J103.3, J104.2, J104.4, J108.2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
- removed net 3.3V7: C124.1, C126.1, C127.1, C131.1, C132.1, D43.A, D44.A, D48.A, J113.3A, J113.3B, J114.2, J114.4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
- removed net 3.3V8: C141.1, C143.1, C144.1, C148.1, C149.1, D49.A, D50.A, D54.A, J129.3A, J129.3B, J130.2, J130.4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
- removed net 3.3V9: C158.1, C160.1, C161.1, C165.1, C166.1, D55.A, D56.A, D60.A, J145.3A, J145.3B, J146.2, J146.4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
- removed net 5V10: C184.1, J162.5, J168.5, J175.2, JP154.2, U64.1, U64.3
- removed net 5V11: C201.1, J178.5, J184.5, J191.2, JP168.2, U70.1, U70.3
- removed net 5V4: C82.1, J66.5, J72.5, J79.2, JP70.2, U28.1, U28.3
- removed net 5V5: C99.1, J82.5, J88.5, J95.2, JP84.2, U34.1, U34.3
- removed net 5V6: C116.1, J104.5, J111.2, J98.5, JP98.2, U40.1, U40.3
- removed net 5V7: C133.1, J114.5, J120.5, J127.2, JP112.2, U46.1, U46.3
- removed net 5V8: C150.1, J130.5, J136.5, J143.2, JP126.2, U52.1, U52.3
- removed net 5V9: C167.1, J146.5, J152.5, J159.2, JP140.2, U58.1, U58.3
- removed net 5V_CHG10: C186.1, D65.A, Q140.4, Q141.2, Q142.4, Q143.2, U65.4
- removed net 5V_CHG11: C203.1, D71.A, Q153.4, Q154.2, Q155.4, Q156.2, U71.4
- removed net 5V_CHG4: C84.1, D29.A, Q62.4, Q63.2, Q64.4, Q65.2, U29.4
- removed net 5V_CHG5: C101.1, D35.A, Q75.4, Q76.2, Q77.4, Q78.2, U35.4
- removed net 5V_CHG6: C118.1, D41.A, Q88.4, Q89.2, Q90.4, Q91.2, U41.4
- removed net 5V_CHG7: C135.1, D47.A, Q101.4, Q102.2, Q103.4, Q104.2, U47.4
- removed net 5V_CHG8: C152.1, D53.A, Q114.4, Q115.2, Q116.4, Q117.2, U53.4
- removed net 5V_CHG9: C169.1, D59.A, Q127.4, Q128.2, Q129.4, Q130.2, U59.4
- removed net 5V_EXT10: C179.+, C180.1, Q136.1, Q137.3, Q142.1, Q143.3, R302.2, R307.1, U63.2, U63.4
- removed net 5V_EXT11: C196.+, C197.1, Q149.1, Q150.3, Q155.1, Q156.3, R331.2, R336.1, U69.2, U69.4
- removed net 5V_EXT4: C77.+, C78.1, Q58.1, Q59.3, Q64.1, Q65.3, R128.2, R133.1, U27.2, U27.4
- removed net 5V_EXT5: C94.+, C95.1, Q71.1, Q72.3, Q77.1, Q78.3, R157.2, R162.1, U33.2, U33.4
- removed net 5V_EXT6: C111.+, C112.1, Q84.1, Q85.3, Q90.1, Q91.3, R186.2, R191.1, U39.2, U39.4
- removed net 5V_EXT7: C128.+, C129.1, Q103.1, Q104.3, Q97.1, Q98.3, R215.2, R220.1, U45.2, U45.4
- removed net 5V_EXT8: C145.+, C146.1, Q110.1, Q111.3, Q116.1, Q117.3, R244.2, R249.1, U51.2, U51.4
- removed net 5V_EXT9: C162.+, C163.1, Q123.1, Q124.3, Q129.1, Q130.3, R273.2, R278.1, U57.2, U57.4
- removed net 5V_MEAS10: J175.1, JP154.1, Q132.4, Q133.2, Q136.4, Q137.2, Q138.4, Q139.2
- removed net 5V_MEAS11: J191.1, JP168.1, Q145.4, Q146.2, Q149.4, Q150.2, Q151.4, Q152.2
- removed net 5V_MEAS4: J79.1, JP70.1, Q54.4, Q55.2, Q58.4, Q59.2, Q60.4, Q61.2
- removed net 5V_MEAS5: J95.1, JP84.1, Q67.4, Q68.2, Q71.4, Q72.2, Q73.4, Q74.2
- removed net 5V_MEAS6: J111.1, JP98.1, Q80.4, Q81.2, Q84.4, Q85.2, Q86.4, Q87.2
- removed net 5V_MEAS7: J127.1, JP112.1, Q100.2, Q93.4, Q94.2, Q97.4, Q98.2, Q99.4
- removed net 5V_MEAS8: J143.1, JP126.1, Q106.4, Q107.2, Q110.4, Q111.2, Q112.4, Q113.2
- removed net 5V_MEAS9: J159.1, JP140.1, Q119.4, Q120.2, Q123.4, Q124.2, Q125.4, Q126.2
- removed net CC10: J69.A5, R120.2
- removed net CC11: J85.B5, R148.2
- removed net CC12: J85.A5, R149.2
- removed net CC13: J101.B5, R177.2
- removed net CC14: J101.A5, R178.2
- removed net CC15: J117.B5, R206.2
- removed net CC16: J117.A5, R207.2
- removed net CC17: J133.B5, R235.2
- removed net CC18: J133.A5, R236.2
- removed net CC19: J149.B5, R264.2
- removed net CC20: J149.A5, R265.2
- removed net CC21: J165.B5, R293.2
- removed net CC22: J165.A5, R294.2
- removed net CC23: J181.B5, R322.2
- removed net CC24: J181.A5, R323.2
- removed net CC9: J69.B5, R119.2
- removed net D+10: J165.A6, J165.B6, J166.D+, U61.5
- removed net D+11: J181.A6, J181.B6, J182.D+, U67.5
- removed net D+4: J69.A6, J69.B6, J70.D+, U25.5
- removed net D+5: J85.A6, J85.B6, J86.D+, U31.5
- removed net D+6: J101.A6, J101.B6, J102.D+, U37.5
- removed net D+7: J117.A6, J117.B6, J118.D+, U43.5
- removed net D+8: J133.A6, J133.B6, J134.D+, U49.5
- removed net D+9: J149.A6, J149.B6, J150.D+, U55.5
- removed net D-10: J165.A7, J165.B7, J166.D-, U61.6
- removed net D-11: J181.A7, J181.B7, J182.D-, U67.6
- removed net D-4: J69.A7, J69.B7, J70.D-, U25.6
- removed net D-5: J85.A7, J85.B7, J86.D-, U31.6
- removed net D-6: J101.A7, J101.B7, J102.D-, U37.6
- removed net D-7: J117.A7, J117.B7, J118.D-, U43.6
- removed net D-8: J133.A7, J133.B7, J134.D-, U49.6
- removed net D-9: J149.A7, J149.B7, J150.D-, U55.6
- removed net ESP32_10: Q131.3, S22.3, S22.4, U62.25
- removed net ESP32_11: Q144.3, S24.3, S24.4, U68.25
- removed net ESP32_4: Q53.3, S10.3, S10.4, U26.25
- removed net ESP32_5: Q66.3, S12.3, S12.4, U32.25
- removed net ESP32_6: Q79.3, S14.3, S14.4, U38.25
- removed net ESP32_7: Q92.3, S16.3, S16.4, U44.25
- removed net ESP32_8: Q105.3, S18.3, S18.4, U50.25
- removed net ESP32_9: Q118.3, S20.3, S20.4, U56.25
- removed net ESP32_ADC24: J68.6, J73.6, U26.4
- removed net ESP32_ADC25: J68.5, J73.5, U26.5
- removed net ESP32_ADC26: J68.4, J73.4, U26.6
- removed net ESP32_ADC27: J68.3, J73.3, U26.7
- removed net ESP32_ADC28: J68.1, J73.1, U26.9
- removed net ESP32_ADC29: J68.2, J73.2, U26.8
- removed net ESP32_ADC30: J84.6, J89.6, U32.4
- removed net ESP32_ADC31: J84.5, J89.5, U32.5
- removed net ESP32_ADC32: J84.4, J89.4, U32.6
- removed net ESP32_ADC33: J84.3, J89.3, U32.7
- removed net ESP32_ADC34: J84.1, J89.1, U32.9
- removed net ESP32_ADC35: J84.2, J89.2, U32.8
- removed net ESP32_ADC36: J100.6, J105.6, U38.4
- removed net ESP32_ADC37: J100.5, J105.5, U38.5
- removed net ESP32_ADC38: J100.4, J105.4, U38.6
- removed net ESP32_ADC39: J100.3, J105.3, U38.7
- removed net ESP32_ADC40: J100.1, J105.1, U38.9
- removed net ESP32_ADC41: J100.2, J105.2, U38.8
- removed net ESP32_ADC42: J116.6, J121.6, U44.4
- removed net ESP32_ADC43: J116.5, J121.5, U44.5
- removed net ESP32_ADC44: J116.4, J121.4, U44.6
- removed net ESP32_ADC45: J116.3, J121.3, U44.7
- removed net ESP32_ADC46: J116.1, J121.1, U44.9
- removed net ESP32_ADC47: J116.2, J121.2, U44.8
- removed net ESP32_ADC48: J132.6, J137.6, U50.4
- removed net ESP32_ADC49: J132.5, J137.5, U50.5
- removed net ESP32_ADC50: J132.4, J137.4, U50.6
- removed net ESP32_ADC51: J132.3, J137.3, U50.7
- removed net ESP32_ADC52: J132.1, J137.1, U50.9
- removed net ESP32_ADC53: J132.2, J137.2, U50.8
- removed net ESP32_ADC54: J148.6, J153.6, U56.4
- removed net ESP32_ADC55: J148.5, J153.5, U56.5
- removed net ESP32_ADC56: J148.4, J153.4, U56.6
- removed net ESP32_ADC57: J148.3, J153.3, U56.7
- removed net ESP32_ADC58: J148.1, J153.1, U56.9
- removed net ESP32_ADC59: J148.2, J153.2, U56.8
- removed net ESP32_ADC60: J164.6, J169.6, U62.4
- removed net ESP32_ADC61: J164.5, J169.5, U62.5
- removed net ESP32_ADC62: J164.4, J169.4, U62.6
- removed net ESP32_ADC63: J164.3, J169.3, U62.7
- removed net ESP32_ADC64: J164.1, J169.1, U62.9
- removed net ESP32_ADC65: J164.2, J169.2, U62.8
- removed net ESP32_ADC66: J180.6, J185.6, U68.4
- removed net ESP32_ADC67: J180.5, J185.5, U68.5
- removed net ESP32_ADC68: J180.4, J185.4, U68.6
- removed net ESP32_ADC69: J180.3, J185.3, U68.7
- removed net ESP32_ADC70: J180.1, J185.1, U68.9
- removed net ESP32_ADC71: J180.2, J185.2, U68.8
- removed net ESP32_EN10: C176.1, J162.3, J168.3, Q131.6, R297.1, S21.3, S21.4, U62.3
- removed net ESP32_EN11: C193.1, J178.3, J184.3, Q144.6, R326.1, S23.3, S23.4, U68.3
- removed net ESP32_EN4: C74.1, J66.3, J72.3, Q53.6, R123.1, S9.3, S9.4, U26.3
- removed net ESP32_EN5: C91.1, J82.3, J88.3, Q66.6, R152.1, S11.3, S11.4, U32.3
- removed net ESP32_EN6: C108.1, J104.3, J98.3, Q79.6, R181.1, S13.3, S13.4, U38.3
- removed net ESP32_EN7: C125.1, J114.3, J120.3, Q92.6, R210.1, S15.3, S15.4, U44.3
- removed net ESP32_EN8: C142.1, J130.3, J136.3, Q105.6, R239.1, S17.3, S17.4, U50.3
- removed net ESP32_EN9: C159.1, J146.3, J152.3, Q118.6, R268.1, S19.3, S19.4, U56.3
- removed net ESP32_GPIO12_TDI10: J171.8, TP11.1, U62.14
- removed net ESP32_GPIO12_TDI11: J187.8, TP12.1, U68.14
- removed net ESP32_GPIO12_TDI4: J75.8, TP5.1, U26.14
- removed net ESP32_GPIO12_TDI5: J91.8, TP6.1, U32.14
- removed net ESP32_GPIO12_TDI6: J107.8, TP7.1, U38.14
- removed net ESP32_GPIO12_TDI7: J123.8, TP8.1, U44.14
- removed net ESP32_GPIO12_TDI8: J139.8, TP9.1, U50.14
- removed net ESP32_GPIO12_TDI9: J155.8, TP10.1, U56.14
- removed net ESP32_GPIO13_HDR10: J163.4, J170.4, JP151.2
- removed net ESP32_GPIO13_HDR11: J179.4, J186.4, JP165.2
- removed net ESP32_GPIO13_HDR4: J67.4, J74.4, JP67.2
- removed net ESP32_GPIO13_HDR5: J83.4, J90.4, JP81.2
- removed net ESP32_GPIO13_HDR6: J106.4, J99.4, JP95.2
- removed net ESP32_GPIO13_HDR7: J115.4, J122.4, JP109.2
- removed net ESP32_GPIO13_HDR8: J131.4, J138.4, JP123.2
- removed net ESP32_GPIO13_HDR9: J147.4, J154.4, JP137.2
- removed net ESP32_GPIO13_TCK10: J171.4, JP151.1, U62.16
- removed net ESP32_GPIO13_TCK11: J187.4, JP165.1, U68.16
- removed net ESP32_GPIO13_TCK4: J75.4, JP67.1, U26.16
- removed net ESP32_GPIO13_TCK5: J91.4, JP81.1, U32.16
- removed net ESP32_GPIO13_TCK6: J107.4, JP95.1, U38.16
- removed net ESP32_GPIO13_TCK7: J123.4, JP109.1, U44.16
- removed net ESP32_GPIO13_TCK8: J139.4, JP123.1, U50.16
- removed net ESP32_GPIO13_TCK9: J155.4, JP137.1, U56.16
- removed net ESP32_GPIO14_HDR10: J163.5, J170.5, JP152.2
- removed net ESP32_GPIO14_HDR11: J179.5, J186.5, JP166.2
- removed net ESP32_GPIO14_HDR4: J67.5, J74.5, JP68.2
- removed net ESP32_GPIO14_HDR5: J83.5, J90.5, JP82.2
- removed net ESP32_GPIO14_HDR6: J106.5, J99.5, JP96.2
- removed net ESP32_GPIO14_HDR7: J115.5, J122.5, JP110.2
- removed net ESP32_GPIO14_HDR8: J131.5, J138.5, JP124.2
- removed net ESP32_GPIO14_HDR9: J147.5, J154.5, JP138.2
- removed net ESP32_GPIO14_TMS10: J171.2, JP152.1, U62.13
- removed net ESP32_GPIO14_TMS11: J187.2, JP166.1, U68.13
- removed net ESP32_GPIO14_TMS4: J75.2, JP68.1, U26.13
- removed net ESP32_GPIO14_TMS5: J91.2, JP82.1, U32.13
- removed net ESP32_GPIO14_TMS6: J107.2, JP96.1, U38.13
- removed net ESP32_GPIO14_TMS7: J123.2, JP110.1, U44.13
- removed net ESP32_GPIO14_TMS8: J139.2, JP124.1, U50.13
- removed net ESP32_GPIO14_TMS9: J155.2, JP138.1, U56.13
- removed net ESP32_GPIO15_TDO10: J171.6, U62.23
- removed net ESP32_GPIO15_TDO11: J187.6, U68.23
- removed net ESP32_GPIO15_TDO4: J75.6, U26.23
- removed net ESP32_GPIO15_TDO5: J91.6, U32.23
- removed net ESP32_GPIO15_TDO6: J107.6, U38.23
- removed net ESP32_GPIO15_TDO7: J123.6, U44.23
- removed net ESP32_GPIO15_TDO8: J139.6, U50.23
- removed net ESP32_GPIO15_TDO9: J155.6, U56.23
- removed net ESP32_GPIO18_SCK10: D63.A, J161.5A, J161.5B, J167.5, J173.5, U62.30
- removed net ESP32_GPIO18_SCK11: D69.A, J177.5A, J177.5B, J183.5, J189.5, U68.30
- removed net ESP32_GPIO18_SCK4: D27.A, J65.5A, J65.5B, J71.5, J77.5, U26.30
- removed net ESP32_GPIO18_SCK5: D33.A, J81.5A, J81.5B, J87.5, J93.5, U32.30
- removed net ESP32_GPIO18_SCK6: D39.A, J103.5, J109.5, J97.5A, J97.5B, U38.30
- removed net ESP32_GPIO18_SCK7: D45.A, J113.5A, J113.5B, J119.5, J125.5, U44.30
- removed net ESP32_GPIO18_SCK8: D51.A, J129.5A, J129.5B, J135.5, J141.5, U50.30
- removed net ESP32_GPIO18_SCK9: D57.A, J145.5A, J145.5B, J151.5, J157.5, U56.30
- removed net ESP32_GPIO19_POCI10: J161.6A, J161.6B, J167.6, J173.7, U62.31
- removed net ESP32_GPIO19_POCI11: J177.6A, J177.6B, J183.6, J189.7, U68.31
- removed net ESP32_GPIO19_POCI4: J65.6A, J65.6B, J71.6, J77.7, U26.31
- removed net ESP32_GPIO19_POCI5: J81.6A, J81.6B, J87.6, J93.7, U32.31
- removed net ESP32_GPIO19_POCI6: J103.6, J109.7, J97.6A, J97.6B, U38.31
- removed net ESP32_GPIO19_POCI7: J113.6A, J113.6B, J119.6, J125.7, U44.31
- removed net ESP32_GPIO19_POCI8: J129.6A, J129.6B, J135.6, J141.7, U50.31
- removed net ESP32_GPIO19_POCI9: J145.6A, J145.6B, J151.6, J157.7, U56.31
- removed net ESP32_GPIO23_PICO10: J161.7A, J161.7B, J167.7, J173.3, U62.37
- removed net ESP32_GPIO23_PICO11: J177.7A, J177.7B, J183.7, J189.3, U68.37
- removed net ESP32_GPIO23_PICO4: J65.7A, J65.7B, J71.7, J77.3, U26.37
- removed net ESP32_GPIO23_PICO5: J81.7A, J81.7B, J87.7, J93.3, U32.37
- removed net ESP32_GPIO23_PICO6: J103.7, J109.3, J97.7A, J97.7B, U38.37
- removed net ESP32_GPIO23_PICO7: J113.7A, J113.7B, J119.7, J125.3, U44.37
- removed net ESP32_GPIO23_PICO8: J129.7A, J129.7B, J135.7, J141.3, U50.37
- removed net ESP32_GPIO23_PICO9: J145.7A, J145.7B, J151.7, J157.3, U56.37
- removed net ESP32_GPIO29: U26.24
- removed net ESP32_GPIO30: J67.3, J74.3, JP66.2, U26.26
- removed net ESP32_GPIO31: J67.7, J74.7, U26.28
- removed net ESP32_GPIO32: J67.8, J74.8, U26.10
- removed net ESP32_GPIO33: J65.10A, J65.10B, J71.10, U26.11
- removed net ESP32_GPIO34: J65.9A, J65.9B, J71.9, U26.12
- removed net ESP32_GPIO35: J67.6, J74.6, U26.27
- removed net ESP32_GPIO36: U32.24
- removed net ESP32_GPIO37: J83.3, J90.3, JP80.2, U32.26
- removed net ESP32_GPIO38: J83.7, J90.7, U32.28
- removed net ESP32_GPIO39: J83.8, J90.8, U32.10
- removed net ESP32_GPIO40: J81.10A, J81.10B, J87.10, U32.11
- removed net ESP32_GPIO41: J81.9A, J81.9B, J87.9, U32.12
- removed net ESP32_GPIO42: J83.6, J90.6, U32.27
- removed net ESP32_GPIO43: U38.24
- removed net ESP32_GPIO44: J106.3, J99.3, JP94.2, U38.26
- removed net ESP32_GPIO45: J106.7, J99.7, U38.28
- removed net ESP32_GPIO46: J106.8, J99.8, U38.10
- removed net ESP32_GPIO47: J103.10, J97.10A, J97.10B, U38.11
- removed net ESP32_GPIO48: J103.9, J97.9A, J97.9B, U38.12
- removed net ESP32_GPIO49: J106.6, J99.6, U38.27
- removed net ESP32_GPIO50: U44.24
- removed net ESP32_GPIO51: J115.3, J122.3, JP108.2, U44.26
- removed net ESP32_GPIO52: J115.7, J122.7, U44.28
- removed net ESP32_GPIO53: J115.8, J122.8, U44.10
- removed net ESP32_GPIO54: J113.10A, J113.10B, J119.10, U44.11
- removed net ESP32_GPIO55: J113.9A, J113.9B, J119.9, U44.12
- removed net ESP32_GPIO56: J115.6, J122.6, U44.27
- removed net ESP32_GPIO57: U50.24
- removed net ESP32_GPIO58: J131.3, J138.3, JP122.2, U50.26
- removed net ESP32_GPIO59: J131.7, J138.7, U50.28
- removed net ESP32_GPIO5_!CS!10: J161.8A, J161.8B, J167.8, J173.2, U62.29
- removed net ESP32_GPIO5_!CS!11: J177.8A, J177.8B, J183.8, J189.2, U68.29
- removed net ESP32_GPIO5_!CS!4: J65.8A, J65.8B, J71.8, J77.2, U26.29
- removed net ESP32_GPIO5_!CS!5: J81.8A, J81.8B, J87.8, J93.2, U32.29
- removed net ESP32_GPIO5_!CS!6: J103.8, J109.2, J97.8A, J97.8B, U38.29
- removed net ESP32_GPIO5_!CS!7: J113.8A, J113.8B, J119.8, J125.2, U44.29
- removed net ESP32_GPIO5_!CS!8: J129.8A, J129.8B, J135.8, J141.2, U50.29
- removed net ESP32_GPIO5_!CS!9: J145.8A, J145.8B, J151.8, J157.2, U56.29
- removed net ESP32_GPIO60: J131.8, J138.8, U50.10
- removed net ESP32_GPIO61: J129.10A, J129.10B, J135.10, U50.11
- removed net ESP32_GPIO62: J129.9A, J129.9B, J135.9, U50.12
- removed net ESP32_GPIO63: J131.6, J138.6, U50.27
- removed net ESP32_GPIO64: U56.24
- removed net ESP32_GPIO65: J147.3, J154.3, JP136.2, U56.26
- removed net ESP32_GPIO66: J147.7, J154.7, U56.28
- removed net ESP32_GPIO67: J147.8, J154.8, U56.10
- removed net ESP32_GPIO68: J145.10A, J145.10B, J151.10, U56.11
- removed net ESP32_GPIO69: J145.9A, J145.9B, J151.9, U56.12
- removed net ESP32_GPIO70: J147.6, J154.6, U56.27
- removed net ESP32_GPIO71: U62.24
- removed net ESP32_GPIO72: J163.3, J170.3, JP150.2, U62.26
- removed net ESP32_GPIO73: J163.7, J170.7, U62.28
- removed net ESP32_GPIO74: J163.8, J170.8, U62.10
- removed net ESP32_GPIO75: J161.10A, J161.10B, J167.10, U62.11
- removed net ESP32_GPIO76: J161.9A, J161.9B, J167.9, U62.12
- removed net ESP32_GPIO77: J163.6, J170.6, U62.27
- removed net ESP32_GPIO78: U68.24
- removed net ESP32_GPIO79: J179.3, J186.3, JP164.2, U68.26
- removed net ESP32_GPIO80: J179.7, J186.7, U68.28
- removed net ESP32_GPIO81: J179.8, J186.8, U68.10
- removed net ESP32_GPIO82: J177.10A, J177.10B, J183.10, U68.11
- removed net ESP32_GPIO83: J177.9A, J177.9B, J183.9, U68.12
- removed net ESP32_GPIO84: J179.6, J186.6, U68.27
- removed net ESP32_RXD10: J163.1, J170.1, R291.1, U61.2, U62.34
- removed net ESP32_RXD11: J179.1, J186.1, R320.1, U67.2, U68.34
- removed net ESP32_RXD4: J67.1, J74.1, R117.1, U25.2, U26.34
- removed net ESP32_RXD5: J83.1, J90.1, R146.1, U31.2, U32.34
- removed net ESP32_RXD6: J106.1, J99.1, R175.1, U37.2, U38.34
- removed net ESP32_RXD7: J115.1, J122.1, R204.1, U43.2, U44.34
- removed net ESP32_RXD8: J131.1, J138.1, R233.1, U49.2, U50.34
- removed net ESP32_RXD9: J147.1, J154.1, R262.1, U55.2, U56.34
- removed net ESP32_SCL10: J161.1A, J161.1B, J167.1, J172.4, R299.1, U62.36, U66.7
- removed net ESP32_SCL11: J177.1A, J177.1B, J183.1, J188.4, R328.1, U68.36, U72.7
- removed net ESP32_SCL4: J65.1A, J65.1B, J71.1, J76.4, R125.1, U26.36, U30.7
- removed net ESP32_SCL5: J81.1A, J81.1B, J87.1, J92.4, R154.1, U32.36, U36.7
- removed net ESP32_SCL6: J103.1, J108.4, J97.1A, J97.1B, R183.1, U38.36, U42.7
- removed net ESP32_SCL7: J113.1A, J113.1B, J119.1, J124.4, R212.1, U44.36, U48.7
- removed net ESP32_SCL8: J129.1A, J129.1B, J135.1, J140.4, R241.1, U50.36, U54.7
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Routing:
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- removed copper zone on layer 15, net 3.3V10
- removed copper zone on layer 15, net 3.3V11
- removed copper zone on layer 15, net 3.3V4
- removed copper zone on layer 15, net 3.3V5
- removed copper zone on layer 15, net 3.3V6
- removed copper zone on layer 15, net 3.3V7
- removed copper zone on layer 15, net 3.3V8
- removed copper zone on layer 15, net 3.3V9
- removed copper zone on layer 1, net 5V_EXT10
- removed copper zone on layer 1, net 5V_EXT11
- removed copper zone on layer 1, net 5V_EXT4
- removed copper zone on layer 1, net 5V_EXT5
- removed copper zone on layer 1, net 5V_EXT6
- removed copper zone on layer 1, net 5V_EXT7
- removed copper zone on layer 1, net 5V_EXT8
- removed copper zone on layer 1, net 5V_EXT9
- removed copper zone on layer 1, net GND10
- removed copper zone on layer 16, net GND10
- removed copper zone on layer 2, net GND10
- removed copper zone on layer 1, net GND12
- removed copper zone on layer 16, net GND12
- removed copper zone on layer 2, net GND12
- removed copper zone on layer 1, net GND14
- removed copper zone on layer 16, net GND14
- removed copper zone on layer 2, net GND14
- removed copper zone on layer 1, net GND16
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Other:
- board size 246.1 x 248.9 mm -> 172.2 x 137.9 mm
