File: production/SparkFun_IoT_RedBoard-ESP32-Panel.brd (EAGLE design)
At the start: 400.1 x 131.1 mm, 2336 parts, among them J1 5.5x2.1mm Barrel, J102 QWIIC_RIGHT_ANGLE, J103 MICRO-SD-PUSH-PUSH-EXT-PIN, J104 5.5x2.1mm Barrel, J110 USB-C, J111 USB_SOLDER_PADS, J112 M10NO_SILK, J117 QWIIC_RIGHT_ANGLE, J118 MICRO-SD-PUSH-PUSH-EXT-PIN, J119 5.5x2.1mm Barrel, J125 USB-C, J126 USB_SOLDER_PADS, J127 M10NO_SILK, J13 QWIIC_RIGHT_ANGLE, J132 QWIIC_RIGHT_ANGLE, J133 MICRO-SD-PUSH-PUSH-EXT-PIN, J134 5.5x2.1mm Barrel, J140 USB-C, J141 USB_SOLDER_PADS, J142 M10NO_SILK, J147 QWIIC_RIGHT_ANGLE, J148 MICRO-SD-PUSH-PUSH-EXT-PIN, J149 5.5x2.1mm Barrel, J15 MICRO-SD-PUSH-PUSH-EXT-PIN, J2 USB-C, J20 USB-C, J21 USB_SOLDER_PADS, J22 M10NO_SILK, J27 QWIIC_RIGHT_ANGLE, J28 MICRO-SD-PUSH-PUSH-EXT-PIN, J29 5.5x2.1mm Barrel, J3 USB_SOLDER_PADS, J35 USB-C, J36 USB_SOLDER_PADS, J37 M10NO_SILK, J42 QWIIC_RIGHT_ANGLE, J43 MICRO-SD-PUSH-PUSH-EXT-PIN, J44 5.5x2.1mm Barrel, J5 M10NO_SILK, J50 USB-C, J51 USB_SOLDER_PADS, J52 M10NO_SILK, J57 QWIIC_RIGHT_ANGLE, J58 MICRO-SD-PUSH-PUSH-EXT-PIN, J59 5.5x2.1mm Barrel, J65 USB-C, J66 USB_SOLDER_PADS, J67 M10NO_SILK, J72 QWIIC_RIGHT_ANGLE, J73 MICRO-SD-PUSH-PUSH-EXT-PIN, J74 5.5x2.1mm Barrel, J80 USB-C, J81 USB_SOLDER_PADS, J82 M10NO_SILK, J87 QWIIC_RIGHT_ANGLE, J88 MICRO-SD-PUSH-PUSH-EXT-PIN, J89 5.5x2.1mm Barrel, J95 USB-C, J96 USB_SOLDER_PADS, J97 M10NO_SILK, Q1 MBT3904DW1T1, Q100 20V/4.2A/52mΩ/1.4W, Q102 20V/4.2A/52mΩ/1.4W, Q104 20V/4.2A/52mΩ/1.4W, Q105 MBT3904DW1T1, Q107 20V/4.2A/52mΩ/1.4W, Q109 20V/4.2A/52mΩ/1.4W, Q11 20V/4.2A/52mΩ/1.4W, Q111 20V/4.2A/52mΩ/1.4W, Q113 20V/4.2A/52mΩ/1.4W, Q115 20V/4.2A/52mΩ/1.4W, Q117 20V/4.2A/52mΩ/1.4W, Q118 MBT3904DW1T1, Q120 20V/4.2A/52mΩ/1.4W, Q122 20V/4.2A/52mΩ/1.4W, Q124 20V/4.2A/52mΩ/1.4W, Q126 20V/4.2A/52mΩ/1.4W, Q128 20V/4.2A/52mΩ/1.4W, Q13 20V/4.2A/52mΩ/1.4W, Q130 20V/4.2A/52mΩ/1.4W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

Commit message: Update panel with fiducials on top/bottom
Parts:
- moved E$5 22.8 mm to (12.7, -2.10)
- moved E$6 22.8 mm to (12.7, -2.10)
- moved E$1 21.7 mm to (12.7, 119.4)
- moved E$2 21.7 mm to (12.7, 119.4)
- moved E$3 6.03 mm to (373.1, 119.4)
- moved E$4 6.03 mm to (373.1, 119.4)
Changed lines of the file:
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@@
 <layers>
 <layer number="1" name="Top" color="4" fill="1" visible="yes" active="yes"/>
+<layer number="2" name="Route2" color="16" fill="1" visible="no" active="yes"/>
+<layer number="15" name="Route15" color="23" fill="1" visible="no" active="yes"/>
 <layer number="16" name="Bottom" color="1" fill="1" visible="yes" active="yes"/>
 <layer number="17" name="Pads" color="2" fill="1" visible="yes" active="yes"/>
@@
 <element name="U$1119" library="output" package="#LED_DO#1" value="" x="340.4616" y="68.4784" smashed="yes" rot="MR0"/>
 <element name="U$1120" library="output" package="#NC#LED_DO#0" value="" x="327.66" y="60.706" smashed="yes" rot="MR90"/>
-<element name="E$1" library="SparkFun-Aesthetics" package="FIDUCIAL-1X2" value="" x="-8.46581875" y="114.681" smashed="yes"/>
-<element name="E$2" library="SparkFun-Aesthetics" package="FIDUCIAL-1X2" value="" x="-8.46581875" y="114.681" smashed="yes" rot="MR0"/>
-<element name="E$3" library="SparkFun-Aesthetics" package="FIDUCIAL-1X2" value="" x="376.76581875" y="114.681" smashed="yes"/>
-<element name="E$4" library="SparkFun-Aesthetics" package="FIDUCIAL-1X2" value="" x="376.76581875" y="114.681" smashed="yes" rot="MR0"/>
-<element name="E$5" library="SparkFun-Retired" package="FIDUCIAL-1.5X3" value="" x="-8.46581875" y="6.35" smashed="yes"/>
-<element name="E$6" library="SparkFun-Retired" package="FIDUCIAL-1.5X3" value="" x="-8.46581875" y="6.35" smashed="yes" rot="MR0"/>
+<element name="E$1" library="SparkFun-Aesthetics" package="FIDUCIAL-1X2" value="" x="12.7" y="119.4435" smashed="yes"/>
+<element name="E$2" library="SparkFun-Aesthetics" package="FIDUCIAL-1X2" value="" x="12.7" y="119.4435" smashed="yes" rot="MR0"/>
+<element name="E$3" library="SparkFun-Aesthetics" package="FIDUCIAL-1X2" value="" x="373.0625" y="119.4435" smashed="yes"/>
+<element name="E$4" library="SparkFun-Aesthetics" package="FIDUCIAL-1X2" value="" x="373.0625" y="119.4435" smashed="yes" rot="MR0"/>
+<element name="E$5" library="SparkFun-Retired" package="FIDUCIAL-1.5X3" value="" x="12.7" y="-2.0955" smashed="yes"/>
+<element name="E$6" library="SparkFun-Retired" package="FIDUCIAL-1.5X3" value="" x="12.7" y="-2.0955" smashed="yes" rot="MR0"/>
 </elements>
 <signals>
@@
 <wire x1="45.593" y1="27.94" x2="43.04" y2="29.845" width="0" layer="19" extent="1-1"/>
 <wire x1="48.3616" y1="28.5496" x2="45.593" y2="27.94" width="0" layer="19" extent="1-1"/>
-<wire x1="50.546" y1="22.733" x2="48.3616" y2="21.6916" width="0" layer="19" extent="1-15"/>
+<wire x1="50.546" y1="22.733" x2="47.752" y2="21.082" width="0" layer="19" extent="1-1"/>
 <wire x1="51.859" y1="23.816" x2="50.546" y2="22.733" width="0" layer="19" extent="1-1"/>
 <wire x1="51.849" y1="25.646" x2="51.859" y2="23.816" width="0" layer="19" extent="1-1"/>
@@
 <wire x1="120.523" y1="27.94" x2="117.97" y2="29.845" width="0" layer="19" extent="1-1"/>
 <wire x1="123.2916" y1="28.5496" x2="120.523" y2="27.94" width="0" layer="19" extent="1-1"/>
-<wire x1="125.476" y1="22.733" x2="123.2916" y2="21.6916" width="0" layer="19" extent="1-15"/>
+<wire x1="125.476" y1="22.733" x2="122.682" y2="21.082" width="0" layer="19" extent="1-1"/>
 <wire x1="126.789" y1="23.816" x2="125.476" y2="22.733" width="0" layer="19" extent="1-1"/>
 <wire x1="126.779" y1="25.646" x2="126.789" y2="23.816" width="0" layer="19" extent="1-1"/>
@@
 <wire x1="195.453" y1="27.94" x2="192.9" y2="29.845" width="0" layer="19" extent="1-1"/>
 <wire x1="198.2216" y1="28.5496" x2="195.453" y2="27.94" width="0" layer="19" extent="1-1"/>
-<wire x1="200.406" y1="22.733" x2="198.2216" y2="21.6916" width="0" layer="19" extent="1-15"/>
+<wire x1="200.406" y1="22.733" x2="197.612" y2="21.082" width="0" layer="19" extent="1-1"/>
 <wire x1="201.719" y1="23.816" x2="200.406" y2="22.733" width="0" layer="19" extent="1-1"/>
 <wire x1="201.709" y1="25.646" x2="201.719" y2="23.816" width="0" layer="19" extent="1-1"/>
@@
 <wire x1="270.383" y1="27.94" x2="267.83" y2="29.845" width="0" layer="19" extent="1-1"/>
 <wire x1="273.1516" y1="28.5496" x2="270.383" y2="27.94" width="0" layer="19" extent="1-1"/>
-<wire x1="275.336" y1="22.733" x2="273.1516" y2="21.6916" width="0" layer="19" extent="1-15"/>
+<wire x1="275.336" y1="22.733" x2="272.542" y2="21.082" width="0" layer="19" extent="1-1"/>
 <wire x1="276.649" y1="23.816" x2="275.336" y2="22.733" width="0" layer="19" extent="1-1"/>
 <wire x1="276.639" y1="25.646" x2="276.649" y2="23.816" width="0" layer="19" extent="1-1"/>
@@
 <wire x1="345.313" y1="27.94" x2="342.76" y2="29.845" width="0" layer="19" extent="1-1"/>
 <wire x1="348.0816" y1="28.5496" x2="345.313" y2="27.94" width="0" layer="19" extent="1-1"/>
-<wire x1="350.266" y1="22.733" x2="348.0816" y2="21.6916" width="0" layer="19" extent="1-15"/>
+<wire x1="350.266" y1="22.733" x2="347.472" y2="21.082" width="0" layer="19" extent="1-1"/>
 <wire x1="351.579" y1="23.816" x2="350.266" y2="22.733" width="0" layer="19" extent="1-1"/>
 <wire x1="351.569" y1="25.646" x2="351.579" y2="23.816" width="0" layer="19" extent="1-1"/>
@@
 <wire x1="45.593" y1="86.868" x2="43.04" y2="88.773" width="0" layer="19" extent="1-1"/>
 <wire x1="48.3616" y1="87.4776" x2="45.593" y2="86.868" width="0" layer="19" extent="1-1"/>
-<wire x1="50.546" y1="81.661" x2="48.3616" y2="80.6196" width="0" layer="19" extent="1-15"/>
+<wire x1="50.546" y1="81.661" x2="47.752" y2="80.01" width="0" layer="19" extent="1-1"/>
 <wire x1="51.859" y1="82.744" x2="50.546" y2="81.661" width="0" layer="19" extent="1-1"/>
 <wire x1="51.849" y1="84.574" x2="51.859" y2="82.744" width="0" layer="19" extent="1-1"/>
@@
 <wire x1="120.523" y1="86.868" x2="117.97" y2="88.773" width="0" layer="19" extent="1-1"/>
 <wire x1="123.2916" y1="87.4776" x2="120.523" y2="86.868" width="0" layer="19" extent="1-1"/>
-<wire x1="125.476" y1="81.661" x2="123.2916" y2="80.6196" width="0" layer="19" extent="1-15"/>
+<wire x1="125.476" y1="81.661" x2="122.682" y2="80.01" width="0" layer="19" extent="1-1"/>
 <wire x1="126.789" y1="82.744" x2="125.476" y2="81.661" width="0" layer="19" extent="1-1"/>
 <wire x1="126.779" y1="84.574" x2="126.789" y2="82.744" width="0" layer="19" extent="1-1"/>
@@
 <wire x1="195.453" y1="86.868" x2="192.9" y2="88.773" width="0" layer="19" extent="1-1"/>
 <wire x1="198.2216" y1="87.4776" x2="195.453" y2="86.868" width="0" layer="19" extent="1-1"/>
-<wire x1="200.406" y1="81.661" x2="198.2216" y2="80.6196" width="0" layer="19" extent="1-15"/>
+<wire x1="200.406" y1="81.661" x2="197.612" y2="80.01" width="0" layer="19" extent="1-1"/>
 <wire x1="201.719" y1="82.744" x2="200.406" y2="81.661" width="0" layer="19" extent="1-1"/>
 <wire x1="201.709" y1="84.574" x2="201.719" y2="82.744" width="0" layer="19" extent="1-1"/>
@@
 <wire x1="270.383" y1="86.868" x2="267.83" y2="88.773" width="0" layer="19" extent="1-1"/>
 <wire x1="273.1516" y1="87.4776" x2="270.383" y2="86.868" width="0" layer="19" extent="1-1"/>
-<wire x1="275.336" y1="81.661" x2="273.1516" y2="80.6196" width="0" layer="19" extent="1-15"/>
+<wire x1="275.336" y1="81.661" x2="272.542" y2="80.01" width="0" layer="19" extent="1-1"/>
 <wire x1="276.649" y1="82.744" x2="275.336" y2="81.661" width="0" layer="19" extent="1-1"/>
 <wire x1="276.639" y1="84.574" x2="276.649" y2="82.744" width="0" layer="19" extent="1-1"/>
@@
 <wire x1="345.313" y1="86.868" x2="342.76" y2="88.773" width="0" layer="19" extent="1-1"/>
 <wire x1="348.0816" y1="87.4776" x2="345.313" y2="86.868" width="0" layer="19" extent="1-1"/>
-<wire x1="350.266" y1="81.661" x2="348.0816" y2="80.6196" width="0" layer="19" extent="1-15"/>
+<wire x1="350.266" y1="81.661" x2="347.472" y2="80.01" width="0" layer="19" extent="1-1"/>
 <wire x1="351.579" y1="82.744" x2="350.266" y2="81.661" width="0" layer="19" extent="1-1"/>
 <wire x1="351.569" y1="84.574" x2="351.579" y2="82.744" width="0" layer="19" extent="1-1"/>

Commit message: Moved panel fiducial and generated gerbers
Parts:
- moved E$3 17.5 mm to (355.6, 119.4)
- moved E$4 17.5 mm to (355.6, 119.4)
Changed lines of the file:
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@@
 <element name="E$1" library="SparkFun-Aesthetics" package="FIDUCIAL-1X2" value="" x="12.7" y="119.4435" smashed="yes"/>
 <element name="E$2" library="SparkFun-Aesthetics" package="FIDUCIAL-1X2" value="" x="12.7" y="119.4435" smashed="yes" rot="MR0"/>
-<element name="E$3" library="SparkFun-Aesthetics" package="FIDUCIAL-1X2" value="" x="373.0625" y="119.4435" smashed="yes"/>
-<element name="E$4" library="SparkFun-Aesthetics" package="FIDUCIAL-1X2" value="" x="373.0625" y="119.4435" smashed="yes" rot="MR0"/>
+<element name="E$3" library="SparkFun-Aesthetics" package="FIDUCIAL-1X2" value="" x="355.6" y="119.4435" smashed="yes"/>
+<element name="E$4" library="SparkFun-Aesthetics" package="FIDUCIAL-1X2" value="" x="355.6" y="119.4435" smashed="yes" rot="MR0"/>
 <element name="E$5" library="SparkFun-Retired" package="FIDUCIAL-1.5X3" value="" x="12.7" y="-2.0955" smashed="yes"/>
 <element name="E$6" library="SparkFun-Retired" package="FIDUCIAL-1.5X3" value="" x="12.7" y="-2.0955" smashed="yes" rot="MR0"/>
